Commit message: Option to specify mesh type

File: simulator/data/irb120/urdf/macros.xacro (robot description, xacro)
@@ -8,5 +8,5 @@
   <xacro:property name="joint_rpy" value="0 0 0" />
   <xacro:property name="joint_type" value="revolute" />
-  <xacro:macro name="irb_120_link" params="name mesh:=0 orig_rpy:=^ orig_xyz:=^ parent:=0 joint_axis:=^ joint_range:=^ joint_xyz:=^ joint_rpy:=^ joint_type:=^ mass:=0 com:=0 com_rpy:=0 inertia:=0">
+  <xacro:macro name="irb_120_link" params="name mesh:=0 orig_rpy:=^ orig_xyz:=^ parent:=0 joint_axis:=^ joint_range:=^ joint_xyz:=^ joint_rpy:=^ joint_type:=^ mass:=0 com:=0 com_rpy:=0 inertia:=0 mesh_type=dae">
     <xacro:if value="${mesh == 0}">
       <xacro:property name="mesh" value="${name}" />
@@ -15,5 +15,5 @@
       <visual>
         <geometry>
-          <mesh filename="../cad/${mesh}.dae"/>
+          <mesh filename="../cad/${mesh}.${mesh_type}"/>
         </geometry>
         <origin rpy="${orig_rpy}" xyz="${orig_xyz}" />
@@ -21,5 +21,5 @@
       <collision>
         <geometry>
-          <mesh filename="../cad/${mesh}.dae"/>
+          <mesh filename="../cad/${mesh}.${mesh_type}"/>
         </geometry>
         <origin rpy="${orig_rpy}" xyz="${orig_xyz}" />

Commit message: Option to specify mesh scale

File: simulator/data/irb120/urdf/macros.xacro (robot description, xacro)
@@ -8,5 +8,5 @@
   <xacro:property name="joint_rpy" value="0 0 0" />
   <xacro:property name="joint_type" value="revolute" />
-  <xacro:macro name="irb_120_link" params="name mesh:=0 orig_rpy:=^ orig_xyz:=^ parent:=0 joint_axis:=^ joint_range:=^ joint_xyz:=^ joint_rpy:=^ joint_type:=^ mass:=0 com:=0 com_rpy:=0 inertia:=0 mesh_type=dae">
+  <xacro:macro name="irb_120_link" params="name mesh:=0 orig_rpy:=^ orig_xyz:=^ parent:=0 joint_axis:=^ joint_range:=^ joint_xyz:=^ joint_rpy:=^ joint_type:=^ mass:=0 com:=0 com_rpy:=0 inertia:=0 mesh_type=dae mesh_scale=1">
     <xacro:if value="${mesh == 0}">
       <xacro:property name="mesh" value="${name}" />
@@ -15,5 +15,5 @@
       <visual>
         <geometry>
-          <mesh filename="../cad/${mesh}.${mesh_type}"/>
+          <mesh filename="../cad/${mesh}.${mesh_type}" scale="${mesh_scale}" />
         </geometry>
         <origin rpy="${orig_rpy}" xyz="${orig_xyz}" />
@@ -21,5 +21,5 @@
       <collision>
         <geometry>
-          <mesh filename="../cad/${mesh}.${mesh_type}"/>
+          <mesh filename="../cad/${mesh}.${mesh_type}" scale="${mesh_scale}" />
         </geometry>
         <origin rpy="${orig_rpy}" xyz="${orig_xyz}" />
