Commit message: Add foundation

File: simulator/data/irb120/urdf/geometry.xacro (robot description, xacro)
@@ -1,4 +1,6 @@
 <?xml version="1.0"?>
 <robot xmlns:xacro="http://ros.org/wiki/xacro">
+  <xacro:property name="orig_foundation_link" value="0 0 0" />
+  <xacro:property name="orig_foundation_joint" value="0 0 0.3" />
   <xacro:property name="orig_base_link" value="0 0 0" />
   <xacro:property name="orig_base_joint" value="0 0 0.166" />

File: simulator/data/irb120/urdf/main.xacro (robot description, xacro)
@@ -5,7 +5,17 @@
   <xacro:include filename="macros.xacro" />
   <xacro:irb_120_link
-    name="base_link"
-    mesh="base"
+    name="foundation"
+    orig_xyz="${orig_foundation_link}"
+    orig_rpy="0 0 0"
+    mesh="foundation"
+    mesh_type="stl"
+    mesh_scale="0.001"
+  />
+  <xacro:irb_120_link
+    name="base"
+    parent="foundation"
     orig_xyz="${orig_base_link}"
+    joint_type="fixed"
+    joint_xyz="${orig_foundation_joint}"
     mass="${mass_base_link}"
     com="${com_base_link}"
@@ -15,5 +25,5 @@
   <xacro:irb_120_link
     name="link1"
-    parent="base_link"
+    parent="base"
     orig_xyz="${orig_link1}"
     joint_axis="0 0 1"
